File: pcb/Micros.sch (KiCad schematic (older format))
At the start: 2 parts, among them J1 Conn_02x08_Top_Bottom

Commit message: Add brigde component.
Parts:
- added C1, C2: 10pF, symbol pspice:CAP
- added C3, C4: 100nF, symbol pspice:CAP
- added CI: LS7366R, symbol Shield_Galileo-rescue:LS7366R-Quanser_2DSFJE_Library
- added Crystal: 30MHz, symbol Device:Crystal
- added Galileo: io8 - io13, symbol Connector_Generic:Conn_01x06
- added Galileo: Pinos, symbol Connector_Generic:Conn_01x02
- added J2: Connector Encoder, symbol Shield_Galileo-rescue:Connector_Encoder-Quanser_2DSFJE_Library
- added PonteH: L298HN, Package_TO_SOT_THT:TO-220-15_P2.54x2.54mm_StaggerOdd_Lead4.58mm_Vertical, symbol Driver_Motor:L298HN
- added R2: 1M, symbol Device:R
Connections:
- net labels added: +5V, GNDREF, MISO, MOSI, SCLK, SS
- wire segments 0 -> 50
Other:
- moved on the sheet: Galileo

Commit message: Update schematic.
Parts:
- removed PonteH: L298HN, Package_TO_SOT_THT:TO-220-15_P2.54x2.54mm_StaggerOdd_Lead4.58mm_Vertical, symbol Driver_Motor:L298HN
- added H-Bridge: LMD18200, Package_TO_SOT_THT:TO-220-11_P3.4x5.08mm_StaggerOdd_Lead4.85mm_Vertical, symbol Driver_Motor:LMD18200
- added Motor: Motor_AC, symbol Motor:Motor_AC
- C3, C4: value 100nF -> 10nF
Connections:
- wire segments 50 -> 86
- no-connect marks 0 -> 24
Changed lines of the file:
@@
 	8300 2100 8300 1800
 $Comp
-L Driver_Motor:L298HN PonteH
-U 1 1 5F2EC224
-P 3550 4650
-F 0 "PonteH" H 3550 5531 50  0000 C CNN
-F 1 "L298HN" H 3550 5440 50  0000 C CNN
-F 2 "Package_TO_SOT_THT:TO-220-15_P2.54x2.54mm_StaggerOdd_Lead4.58mm_Vertical" H 3600 4000 50  0001 L CNN
-F 3 "http://www.st.com/st-web-ui/static/active/en/resource/technical/document/datasheet/CD00000240.pdf" H 3700 4900 50  0001 C CNN
-	1    3550 4650
+L Driver_Motor:LMD18200 H-Bridge
+U 1 1 5F3866DE
+P 3850 4750
+F 0 "H-Bridge" H 3850 5731 50  0000 C CNN
+F 1 "LMD18200" H 3850 5640 50  0000 C CNN
+F 2 "Package_TO_SOT_THT:TO-220-11_P3.4x5.08mm_StaggerOdd_Lead4.85mm_Vertical" H 2400 3400 50  0001 L CNN
+F 3 "http://www.ti.com/lit/ds/symlink/lmd18200.pdf" H 3750 4750 50  0001 C CNN
+	1    3850 4750
+	1    0    0    -1
+$EndComp
+$Comp
+L power:GNDREF #PWR?
+U 1 1 5F3895E3
+P 3850 5850
+F 0 "#PWR?" H 3850 5600 50  0001 C CNN
+F 1 "GNDREF" H 3855 5677 50  0000 C CNN
+F 2 "" H 3850 5850 50  0001 C CNN
+F 3 "" H 3850 5850 50  0001 C CNN
+	1    3850 5850
 	1    0    0    -1
 $EndComp
 Wire Wire Line
-	3550 5500 3550 5350
+	3850 5650 3850 5750
 $Comp
 L pspice:CAP C3
-U 1 1 5F2F5DE3
-P 5250 4600
-F 0 "C3" H 5428 4646 50  0000 L CNN
-F 1 "100nF" H 5428 4555 50  0000 L CNN
-F 2 "" H 5250 4600 50  0001 C CNN
-F 3 "~" H 5250 4600 50  0001 C CNN
-	1    5250 4600
-	1    0    0    -1
-$EndComp
-$Comp
-L pspice:CAP C4
-U 1 1 5F2F9FB7
-P 6000 4600
-F 0 "C4" H 6178 4646 50  0000 L CNN
-F 1 "100nF" H 6178 4555 50  0000 L CNN
-F 2 "" H 6000 4600 50  0001 C CNN
-F 3 "~" H 6000 4600 50  0001 C CNN
-	1    6000 4600
+U 1 1 5F38EF9A
+P 5250 4300
+F 0 "C3" H 5428 4346 50  0000 L CNN
+F 1 "10nF" H 5428 4255 50  0000 L CNN
+F 2 "" H 5250 4300 50  0001 C CNN
+F 3 "~" H 5250 4300 50  0001 C CNN
+	1    5250 4300
 	1    0    0    -1
 $EndComp
 Wire Wire Line
-	3550 5500 5250 5500
+	4550 4150 4700 4150
 Wire Wire Line
-	6000 3750 6000 4350
+	4700 4150 4700 4050
 Wire Wire Line
-	6000 4850 6000 5500
+	4700 4050 5250 4050
 Wire Wire Line
-	3550 3950 3550 3900
+	4550 4450 4700 4450
 Wire Wire Line
-	3550 3900 5250 3900
+	4700 4450 4700 4550
 Wire Wire Line
-	5250 3900 5250 4350
-Wire Wire Line
-	5250 4850 5250 5500
-Connection ~ 5250 5500
-Wire Wire Line
-	5250 5500 6000 5500
+	4700 4550 5250 4550
+Connection ~ 5250 4050
 $Comp
-L power:+5V #PWR?
-U 1 1 5F2FFCD8
-P 3150 3650
-F 0 "#PWR?" H 3150 3500 50  0001 C CNN
-F 1 "+5V" H 3165 3823 50  0000 C CNN
-F 2 "" H 3150 3650 50  0001 C CNN
-F 3 "" H 3150 3650 50  0001 C CNN
-	1    3150 3650
+L pspice:CAP C4
+U 1 1 5F3977D7
+P 5250 4850
+F 0 "C4" H 5428 4896 50  0000 L CNN
+F 1 "10nF" H 5428 4805 50  0000 L CNN
+F 2 "" H 5250 4850 50  0001 C CNN
+F 3 "~" H 5250 4850 50  0001 C CNN
+	1    5250 4850
 	1    0    0    -1
 $EndComp
 Wire Wire Line
-	3650 3950 3900 3950
+	4550 4650 4700 4650
 Wire Wire Line
-	3900 3950 3900 3750
+	4700 4650 4700 4600
 Wire Wire Line
-	3900 3750 6000 3750
+	4700 4600 5250 4600
 Wire Wire Line
-	3150 3650 3150 3900
+	4550 4950 4700 4950
 Wire Wire Line
-	3150 3900 3550 3900
-Connection ~ 3550 3900
+	4700 4950 4700 5100
+Wire Wire Line
+	4700 5100 5250 5100
+$Comp
+L power:PWR_FLAG #FLG?
+U 1 1 5F39B700
+P 3850 3550
+F 0 "#FLG?" H 3850 3625 50  0001 C CNN
+F 1 "PWR_FLAG" H 3850 3723 50  0000 C CNN
+F 2 "" H 3850 3550 50  0001 C CNN
+F 3 "~" H 3850 3550 50  0001 C CNN
+	1    3850 3550
+	1    0    0    -1
+$EndComp
+Wire Wire Line
+	3850 3950 4100 3950
+Wire Wire Line
+	4100 3950 4100 3700
+Wire Wire Line
+	4100 3700 3850 3700
+Wire Wire Line
+	3850 3700 3850 3550
+Wire Wire Line
+	5250 5100 6000 5100
+Connection ~ 5250 5100
+Wire Wire Line
+	5250 4050 6000 4050
+$Comp
+L Motor:Motor_AC Motor
+U 1 1 5F3B10F0
+P 6000 4500
+F 0 "Motor" H 6158 4496 50  0000 L CNN
+F 1 "Motor_AC" H 6158 4405 50  0000 L CNN
+F 2 "" H 6000 4410 50  0001 C CNN
+F 3 "~" H 6000 4410 50  0001 C CNN
+	1    6000 4500
+	1    0    0    -1
+$EndComp
+Wire Wire Line
+	6000 4050 6000 4300
+Wire Wire Line
+	6000 4800 6000 5100
+Text GLabel 2300 4450 0    50   Input ~ 0
+PWM
+Wire Wire Line
+	2300 4450 3150 4450
+Wire Wire Line
+	4550 5150 4800 5150
+Wire Wire Line
+	4800 5150 4800 5750
+Wire Wire Line
+	4800 5750 3850 5750
+Connection ~ 3850 5750
+Wire Wire Line
+	3850 5750 3850 5850
+NoConn ~ 5000 5250
+Wire Wire Line
+	4550 5250 5000 5250
+NoConn ~ 6650 2350
+NoConn ~ 6650 2500
+NoConn ~ 6650 2650
+Wire Wire Line
+	6450 2650 6650 2650
+Wire Wire Line
+	6450 2500 6650 2500
+Wire Wire Line
+	6450 2350 6650 2350
+NoConn ~ 10150 1650
+NoConn ~ 10150 1750
+NoConn ~ 10150 1850
+NoConn ~ 10150 1950
+NoConn ~ 10150 2200
+NoConn ~ 10150 2300
+NoConn ~ 10100 3050
+NoConn ~ 10100 3150
+NoConn ~ 10100 3250
+NoConn ~ 10100 3350
+NoConn ~ 10100 3450
+NoConn ~ 10100 3550
+NoConn ~ 10100 3750
+NoConn ~ 10100 3650
+NoConn ~ 10800 3750
+NoConn ~ 10800 3650
+NoConn ~ 10800 3550
+NoConn ~ 10800 3450
+NoConn ~ 10800 3150
+NoConn ~ 10800 3050
+Wire Wire Line
+	10150 1650 10300 1650
+Wire Wire Line
+	10150 1750 10300 1750
+Wire Wire Line
+	10150 1850 10300 1850
+Wire Wire Line
+	10150 1950 10300 1950
+Wire Wire Line
+	10150 2200 10300 2200
+Wire Wire Line
+	10150 2300 10300 2300
+Wire Wire Line
+	10100 3050 10200 3050
+Wire Wire Line
+	10100 3150 10200 3150
+Wire Wire Line
+	10100 3250 10200 3250
+Wire Wire Line
+	10100 3350 10200 3350
+Wire Wire Line
+	10100 3450 10200 3450
+Wire Wire Line
+	10100 3550 10200 3550
+Wire Wire Line
+	10100 3650 10200 3650
+Wire Wire Line
+	10100 3750 10200 3750
+Wire Wire Line
+	10800 3750 10700 3750
+Wire Wire Line
+	10800 3650 10700 3650
+Wire Wire Line
+	10800 3550 10700 3550
+Wire Wire Line
+	10800 3450 10700 3450
+Wire Wire Line
+	10800 3150 10700 3150
+Wire Wire Line
+	10800 3050 10700 3050
 $EndSCHEMATC

Commit message: Fix motor AC to DC symbol.
Parts:
- removed Motor: Motor_AC, symbol Motor:Motor_AC
- added M1: Motor_DC, symbol Motor:Motor_DC
Changed lines of the file:
@@
 Wire Wire Line
 	5250 4050 6000 4050
-$Comp
-L Motor:Motor_AC Motor
-U 1 1 5F3B10F0
-P 6000 4500
-F 0 "Motor" H 6158 4496 50  0000 L CNN
-F 1 "Motor_AC" H 6158 4405 50  0000 L CNN
-F 2 "" H 6000 4410 50  0001 C CNN
-F 3 "~" H 6000 4410 50  0001 C CNN
-	1    6000 4500
-	1    0    0    -1
-$EndComp
 Wire Wire Line
 	6000 4050 6000 4300
@@
 Wire Wire Line
 	10800 3050 10700 3050
+$Comp
+L Motor:Motor_DC M1
+U 1 1 5F40B5F8
+P 6000 4500
+F 0 "M1" H 6158 4496 50  0000 L CNN
+F 1 "Motor_DC" H 6158 4405 50  0000 L CNN
+F 2 "" H 6000 4410 50  0001 C CNN
+F 3 "~" H 6000 4410 50  0001 C CNN
+	1    6000 4500
+	1    0    0    -1
+$EndComp
 $EndSCHEMATC

Commit message: Add PWM and ENABLE logic to brake the motor.
Parts:
- added Q1, Q2, Q3, Q4: BC817, Package_TO_SOT_SMD:SOT-23, symbol Transistor_BJT:BC817
- added R1, R4 (x2), R7: 10k, symbol Device:R
- added R3, R5, R6: 1k, symbol Device:R
Connections:
- net labels added: 27V, DIRECTION, ENABLE
- wire segments 86 -> 122
Other:
- moved on the sheet: C3, C4, H-Bridge

Commit message: update pcb; add netlist
Parts:
- C1, C2, C3, C4: footprint (none) -> Capacitor_THT:C_Axial_L3.8mm_D2.6mm_P7.50mm_Horizontal
- CI1: renamed from CI; footprint (none) -> Connector_PinHeader_2.54mm:PinHeader_2x07_P2.54mm_Vertical
- Crystal1: renamed from Crystal; footprint (none) -> Crystal:Crystal_HC18-U_Vertical
- Galileo1: renamed from Galileo; footprint (none) -> Connector_PinHeader_2.54mm:PinHeader_1x02_P2.54mm_Vertical
- Galileo2: renamed from Galileo; footprint (none) -> Connector_PinHeader_2.54mm:PinHeader_1x08_P2.54mm_Vertical
- Galileo3: renamed from Galileo; footprint (none) -> Connector_PinHeader_2.54mm:PinHeader_1x06_P2.54mm_Vertical
- J1: footprint (none) -> Connector_PinHeader_2.54mm:PinHeader_2x08_P2.54mm_Vertical
- J2: footprint (none) -> Connector_PinHeader_2.54mm:PinHeader_1x05_P2.54mm_Vertical
- M1: footprint (none) -> TerminalBlock:TerminalBlock_Altech_AK300-2_P5.00mm
- R1, R2, R3, R4, R5, R6, R7: footprint (none) -> Resistor_THT:R_Axial_DIN0204_L3.6mm_D1.6mm_P5.08mm_Horizontal
- R44: renamed from R4; footprint (none) -> Resistor_THT:R_Axial_DIN0204_L3.6mm_D1.6mm_P5.08mm_Horizontal
- renumbered H-Bridge to H-Bridge1
Connections:
- wire segments 122 -> 120
- no-connect marks 24 -> 22
