File: pcb/Micros.sch (KiCad schematic (older format))
At the start: 25 parts, among them J1 Conn_02x08_Top_Bottom, J2 Connector Encoder, M1 Motor_DC, Q1 BC817, Q2 BC817, Q3 BC817, Q4 BC817

Commit message: Fix unconnected pins.
Connections:
- wire segments 122 -> 125
- no-connect marks 24 -> 26
Changed lines of the file:
@@
 Wire Wire Line
 	5450 4700 6050 4700
+NoConn ~ 10150 1250
+Wire Wire Line
+	10150 1250 10300 1250
+NoConn ~ 7850 2450
+Wire Wire Line
+	7850 2450 7750 2450
+Wire Wire Line
+	7750 2450 7750 2300
 $EndSCHEMATC

Commit message: Update the project.
Parts:
- removed Galileo: io0 - io7, symbol Connector_Generic:Conn_01x08
- removed Galileo: io8 - io13, symbol Connector_Generic:Conn_01x06
- removed Galileo: Pinos, symbol Connector_Generic:Conn_01x02
- removed J1: Conn_02x08_Top_Bottom, symbol Connector_Generic:Conn_02x08_Top_Bottom
- removed M1: Motor_DC, symbol Motor:Motor_DC
- removed Q1, Q2, Q3, Q4: BC817, Package_TO_SOT_SMD:SOT-23, symbol Transistor_BJT:BC817
- removed R1, R4 (x2), R7: 10k, symbol Device:R
- removed R5, R6: 1k, symbol Device:R
- added J1: Conn_02x16, symbol Connector_Generic:Conn_02x08_Odd_Even
- added J3: Conn_01x10, symbol Connector_Generic:Conn_01x10
- added J4, J5: Conn_01x08, symbol Connector_Generic:Conn_01x08
- added J6: Conn_Coaxial, symbol Connector:Conn_Coaxial
- added J6: Conn_01x01_Female, symbol Connector:Conn_01x01_Female
- added Q1: BC548, Package_TO_SOT_THT:TO-92_Inline, symbol Transistor_BJT:BC548
- added R2: 0.1R, symbol Device:R
- R3: value 1k -> 10K
- renumbered R2 to R1, H-Bridge to U1, CI to U2
Connections:
- net labels added: #SS, +27V, GND, TH_FLAG
- net labels removed: 27V, DIRECTION, GNDREF, SS
- wire segments 125 -> 106
- no-connect marks 26 -> 32

Commit message: Add NOT port to project.
Parts:
- removed Q1: BC548, Package_TO_SOT_THT:TO-92_Inline, symbol Transistor_BJT:BC548
- added U3: 74AUP1G04, symbol 74xGxx:74AUP1G04
Connections:
- wire segments 106 -> 107
Changed lines of the file:
@@
 Wire Wire Line
 	10800 3050 10700 3050
-Text GLabel 3950 5250 0    50   Input ~ 0
+Text GLabel 3900 5000 0    50   Input ~ 0
 ENABLE
 NoConn ~ 10300 850
@@
 L power:+5V #PWR?
 U 1 1 5F43BC51
-P 4850 4600
-F 0 "#PWR?" H 4850 4450 50  0001 C CNN
-F 1 "+5V" H 4865 4773 50  0000 C CNN
-F 2 "" H 4850 4600 50  0001 C CNN
-F 3 "" H 4850 4600 50  0001 C CNN
-	1    4850 4600
-	1    0    0    -1
-$EndComp
-$Comp
-L power:GND #PWR?
-U 1 1 5F441BC7
-P 4850 5700
-F 0 "#PWR?" H 4850 5450 50  0001 C CNN
-F 1 "GND" H 4855 5527 50  0000 C CNN
-F 2 "" H 4850 5700 50  0001 C CNN
-F 3 "" H 4850 5700 50  0001 C CNN
-	1    4850 5700
+P 4600 4650
+F 0 "#PWR?" H 4600 4500 50  0001 C CNN
+F 1 "+5V" H 4615 4823 50  0000 C CNN
+F 2 "" H 4600 4650 50  0001 C CNN
+F 3 "" H 4600 4650 50  0001 C CNN
+	1    4600 4650
 	1    0    0    -1
 $EndComp
@@
 Wire Wire Line
 	9450 2100 9500 2100
-$Comp
-L Transistor_BJT:BC548 Q1
-U 1 1 5F515402
-P 3950 4700
-F 0 "Q1" H 4141 4746 50  0000 L CNN
-F 1 "BC548" H 4141 4655 50  0000 L CNN
-F 2 "Package_TO_SOT_THT:TO-92_Inline" H 4150 4625 50  0001 L CIN
-F 3 "http://www.fairchildsemi.com/ds/BC/BC547.pdf" H 3950 4700 50  0001 L CNN
-	1    3950 4700
-	1    0    0    -1
-$EndComp
-Wire Wire Line
-	4850 5450 4850 5700
-Wire Wire Line
-	4850 5050 4850 5000
 Wire Wire Line
 	4850 5000 6050 5000
+$Comp
+L 74xGxx:74AUP1G04 U3
+U 1 1 5F540C57
+P 4600 5000
+F 0 "U3" H 4575 5175 50  0000 C CNN
+F 1 "74AUP1G04" H 4575 5176 50  0001 C CNN
+F 2 "" H 4600 5000 50  0001 C CNN
+F 3 "http://www.ti.com/lit/sg/scyt129e/scyt129e.pdf" H 4600 5000 50  0001 C CNN
+	1    4600 5000
+	1    0    0    -1
+$EndComp
+Wire Wire Line
+	3900 5000 4300 5000
+Wire Wire Line
+	4600 4650 4600 4900
+$Comp
+L power:GND #PWR?
+U 1 1 5F553906
+P 4600 5350
+F 0 "#PWR?" H 4600 5100 50  0001 C CNN
+F 1 "GND" H 4605 5177 50  0000 C CNN
+F 2 "" H 4600 5350 50  0001 C CNN
+F 3 "" H 4600 5350 50  0001 C CNN
+	1    4600 5350
+	1    0    0    -1
+$EndComp
+Wire Wire Line
+	4600 5100 4600 5350
 $EndSCHEMATC

Commit message: Update NOT port.
Parts:
- removed U3: 74AUP1G04, symbol 74xGxx:74AUP1G04
- added U3: 74LVC1G04, symbol 74xGxx:74LVC1G04
Changed lines of the file:
@@
 Wire Wire Line
 	4850 5000 6050 5000
-$Comp
-L 74xGxx:74AUP1G04 U3
-U 1 1 5F540C57
-P 4600 5000
-F 0 "U3" H 4575 5175 50  0000 C CNN
-F 1 "74AUP1G04" H 4575 5176 50  0001 C CNN
-F 2 "" H 4600 5000 50  0001 C CNN
-F 3 "http://www.ti.com/lit/sg/scyt129e/scyt129e.pdf" H 4600 5000 50  0001 C CNN
-	1    4600 5000
-	1    0    0    -1
-$EndComp
 Wire Wire Line
 	3900 5000 4300 5000
@@
 Wire Wire Line
 	4600 5100 4600 5350
+$Comp
+L 74xGxx:74LVC1G04 U3
+U 1 1 5F56311C
+P 4600 5000
+F 0 "U3" H 4575 5175 50  0000 C CNN
+F 1 "74LVC1G04" H 4575 5176 50  0001 C CNN
+F 2 "" H 4600 5000 50  0001 C CNN
+F 3 "http://www.ti.com/lit/sg/scyt129e/scyt129e.pdf" H 4600 5000 50  0001 C CNN
+	1    4600 5000
+	1    0    0    -1
+$EndComp
 $EndSCHEMATC

Commit message: Add netlist.
Parts:
- removed J6: Conn_01x01_Female, symbol Connector:Conn_01x01_Female
- removed U2: LS7366R, symbol Shield_Galileo-rescue:LS7366R-Quanser_2DSFJE_Library
- added F1: Fuse, Fuse:Fuse_2010_5025Metric_Pad1.52x2.65mm_HandSolder, symbol Device:Fuse
- added J7: Screw_Terminal_01x02, Connector_PinHeader_2.00mm:PinHeader_1x02_P2.00mm_Vertical, symbol Connector:Screw_Terminal_01x02
- added U2: LS7366R, SOIC14, symbol LS7366R:LS7366R
- C1, C2, C3, C4: footprint (none) -> Capacitor_THT:C_Disc_D3.0mm_W2.0mm_P2.50mm
- Crystal1: renamed from Crystal; footprint (none) -> Crystal:Crystal_HC52-6mm_Vertical
- J1: value Conn_02x16 -> Conn_02x08; footprint (none) -> Connector_PinHeader_2.00mm:PinHeader_2x08_P2.00mm_Vertical
- J2: footprint (none) -> Connector_PinHeader_2.54mm:PinHeader_1x05_P2.54mm_Vertical
- J3: footprint (none) -> Connector_PinHeader_2.00mm:PinHeader_1x10_P2.00mm_Vertical
- J4, J5: footprint (none) -> Connector_PinHeader_2.00mm:PinHeader_1x08_P2.00mm_Vertical
- J6: footprint (none) -> TerminalBlock:TerminalBlock_Altech_AK300-2_P5.00mm
- R1, R2, R3: footprint (none) -> Resistor_THT:R_Axial_DIN0204_L3.6mm_D1.6mm_P5.08mm_Horizontal
- U3: footprint (none) -> Connector_PinHeader_2.00mm:PinHeader_2x03_P2.00mm_Vertical
Connections:
- wire segments 107 -> 106
Other:
- moved on the sheet: C2, J2
