File: pcb/Micros.sch (KiCad schematic (older format))
At the start: 19 parts, among them J1 Conn_02x08, J2 Connector Encoder, J3 Conn_01x10, J4 Conn_01x08, J5 Conn_01x08, J6 Conn_Coaxial, J7 Screw_Terminal_01x02, U1 LMD18200, U2 LS7366R, U3 74LVC1G04

Commit message: Add Gerber files.
Connections:
- net labels added: +27V
- net labels removed: +28V
Changed lines of the file:
@@
 EESchema Schematic File Version 4
-LIBS:Micros-cache
-EELAYER 26 0
+EELAYER 30 0
 EELAYER END
 $Descr A4 11693 8268
@@
 Connection ~ 2400 1850
 $Comp
-L power:+28V #PWR0110
-U 1 1 5F463C7E
+L +27v:+27V #PWR?
+U 1 1 5F54B278
 P 6750 3200
-F 0 "#PWR0110" H 6750 3050 50  0001 C CNN
-F 1 "+28V" H 6765 3373 50  0000 C CNN
+F 0 "#PWR?" H 6750 3050 50  0001 C CNN
+F 1 "+27V" H 6750 3373 50  0000 C CNN
 F 2 "" H 7000 3250 50  0001 C CNN
 F 3 "" H 7000 3250 50  0001 C CNN
@@
 $EndComp
 $Comp
-L power:+28V #PWR0114
-U 1 1 5F46776D
+L +27v:+27V #PWR?
+U 1 1 5F54BCD2
 P 9150 2050
-F 0 "#PWR0114" H 9150 1900 50  0001 C CNN
-F 1 "+28V" H 9165 2223 50  0000 C CNN
+F 0 "#PWR?" H 9150 1900 50  0001 C CNN
+F 1 "+27V" H 9150 2223 50  0000 C CNN
 F 2 "" H 9400 2100 50  0001 C CNN
 F 3 "" H 9400 2100 50  0001 C CNN

Commit message: Ajusta esquemático.
Parts:
- removed J6: Conn_Coaxial, TerminalBlock:TerminalBlock_Altech_AK300-2_P5.00mm, symbol Connector:Conn_Coaxial
- added J6: Screw_Terminal_01x02, TerminalBlock:TerminalBlock_Altech_AK300-2_P5.00mm, symbol Connector:Screw_Terminal_01x02
- F1: value Fuse -> 3A
- J7: footprint Connector_PinHeader_2.00mm:PinHeader_1x02_P2.00mm_Vertical -> TerminalBlock:TerminalBlock_Altech_AK300-2_P5.00mm
Connections:
- net at C4.2, U1.10 (OUTPUT2): now also J6.2 (Pin_2)
- net at C3.1, U1.2 (OUTPUT1): now also J6.1 (Pin_1)
Changed lines of the file:
@@
 P 6750 4700
 F 0 "U1" H 6750 5681 50  0000 L TNN
-F 1 "LMD18200" H 6750 5590 50  0001 L CNN
+F 1 "LMD18200" H 6750 5590 50  0000 L TNN
 F 2 "Package_TO_SOT_THT:TO-220-11_P3.4x5.08mm_StaggerOdd_Lead4.85mm_Vertical" H 5300 3350 50  0001 L CNN
 F 3 "http://www.ti.com/lit/ds/symlink/lmd18200.pdf" H 6650 4700 50  0001 C CNN
@@
 	9500 1450 9500 1350
 Connection ~ 9500 1350
-Wire Wire Line
-	9500 1350 9250 1350
 NoConn ~ 9450 1550
 Wire Wire Line
@@
 Text GLabel 10450 1150 0    50   Output ~ 0
 ENABLE
-$Comp
-L Connector:Conn_Coaxial J6
-U 1 1 5F3E1428
-P 8800 4450
-F 0 "J6" H 8900 4379 50  0000 L CNN
-F 1 "Conn_Coaxial" H 8900 4334 50  0001 L CNN
-F 2 "TerminalBlock:TerminalBlock_Altech_AK300-2_P5.00mm" H 8800 4450 50  0001 C CNN
-F 3 " ~" H 8800 4450 50  0001 C CNN
-	1    8800 4450
-	1    0    0    -1
-$EndComp
 Wire Wire Line
 	8150 4000 8600 4000
@@
 	8600 4000 8600 4450
 Connection ~ 8150 4000
-Wire Wire Line
-	8150 5050 8800 5050
-Wire Wire Line
-	8800 5050 8800 4650
-Connection ~ 8150 5050
 Wire Wire Line
 	5550 4400 5550 4350
@@
 Wire Wire Line
 	5550 4400 6050 4400
-$Comp
-L power:+5V #PWR0112
-U 1 1 5F43BC51
-P 4600 4650
-F 0 "#PWR0112" H 4600 4500 50  0001 C CNN
-F 1 "+5V" H 4615 4823 50  0000 C CNN
-F 2 "" H 4600 4650 50  0001 C CNN
-F 3 "" H 4600 4650 50  0001 C CNN
-	1    4600 4650
-	1    0    0    -1
-$EndComp
 Wire Wire Line
 	5650 4700 6050 4700
@@
 Wire Wire Line
 	3900 5000 4300 5000
-Wire Wire Line
-	4600 4650 4600 4900
-$Comp
-L power:GND #PWR0115
-U 1 1 5F553906
-P 4600 5350
-F 0 "#PWR0115" H 4600 5100 50  0001 C CNN
-F 1 "GND" H 4605 5177 50  0000 C CNN
-F 2 "" H 4600 5350 50  0001 C CNN
-F 3 "" H 4600 5350 50  0001 C CNN
-	1    4600 5350
-	1    0    0    -1
-$EndComp
-Wire Wire Line
-	4600 5100 4600 5350
 $Comp
 L 74xGxx:74LVC1G04 U3
@@
 U 1 1 5F56CD65
 P 6750 3600
-F 0 "F1" H 6810 3600 50  0000 L CNN
-F 1 "Fuse" H 6810 3555 50  0001 L CNN
+F 0 "F1" H 6810 3600 50  0000 L BNN
+F 1 "3A" H 6810 3555 50  0000 L CNN
 F 2 "Fuse:Fuse_2010_5025Metric_Pad1.52x2.65mm_HandSolder" V 6680 3600 50  0001 C CNN
 F 3 "~" H 6750 3600 50  0001 C CNN
@@
 F 0 "J7" H 9730 2096 50  0000 L CNN
 F 1 "Screw_Terminal_01x02" H 9730 2051 50  0001 L CNN
-F 2 "Connector_PinHeader_2.00mm:PinHeader_1x02_P2.00mm_Vertical" H 9650 2150 50  0001 C CNN
+F 2 "TerminalBlock:TerminalBlock_Altech_AK300-2_P5.00mm" H 9650 2150 50  0001 C CNN
 F 3 "~" H 9650 2150 50  0001 C CNN
 	1    9650 2150
@@
 U 1 1 5F48F67C
 P 6250 2050
-F 0 "U2" H 6250 2525 50  0000 C CNN
-F 1 "LS7366R" H 6250 2526 50  0001 C CNN
+F 0 "U2" H 6250 2525 50  0000 C TNN
+F 1 "LS7366R" H 6250 2526 50  0000 C BNN
 F 2 "footNovo:DIP-14_W7.62mm" H 6250 2050 50  0001 L BNN
 F 3 "" H 6250 2050 50  0001 C CNN
@@
 Connection ~ 2400 1850
 $Comp
-L +27v:+27V #PWR?
+L +27v:+27V #PWR0110
 U 1 1 5F54B278
 P 6750 3200
-F 0 "#PWR?" H 6750 3050 50  0001 C CNN
+F 0 "#PWR0110" H 6750 3050 50  0001 C CNN
 F 1 "+27V" H 6750 3373 50  0000 C CNN
 F 2 "" H 7000 3250 50  0001 C CNN
@@
 $EndComp
 $Comp
-L +27v:+27V #PWR?
+L +27v:+27V #PWR0114
 U 1 1 5F54BCD2
 P 9150 2050
-F 0 "#PWR?" H 9150 1900 50  0001 C CNN
+F 0 "#PWR0114" H 9150 1900 50  0001 C CNN
 F 1 "+27V" H 9150 2223 50  0000 C CNN
 F 2 "" H 9400 2100 50  0001 C CNN
@@
 	1    0    0    -1
 $EndComp
+$Comp
+L Connector:Screw_Terminal_01x02 J6
+U 1 1 5F47AB49
+P 8800 4450
+F 0 "J6" H 8880 4396 50  0000 L CNN
+F 1 "Screw_Terminal_01x02" H 8880 4351 50  0001 L CNN
+F 2 "TerminalBlock:TerminalBlock_Altech_AK300-2_P5.00mm" H 8800 4450 50  0001 C CNN
+F 3 "~" H 8800 4450 50  0001 C CNN
+	1    8800 4450
+	1    0    0    -1
+$EndComp
+Wire Wire Line
+	8150 5050 8600 5050
+Wire Wire Line
+	8600 5050 8600 4550
+Connection ~ 8150 5050
+$Comp
+L power:VCC #PWR?
+U 1 1 5F49DD67
+P 8850 1250
+F 0 "#PWR?" H 8850 1100 50  0001 C CNN
+F 1 "VCC" H 8867 1423 50  0000 C CNN
+F 2 "" H 8850 1250 50  0001 C CNN
+F 3 "" H 8850 1250 50  0001 C CNN
+	1    8850 1250
+	1    0    0    -1
+$EndComp
+Wire Wire Line
+	9050 1250 8850 1250
+Connection ~ 9050 1250
+$Comp
+L power:GNDREF #PWR?
+U 1 1 5F4A2B76
+P 9050 1350
+F 0 "#PWR?" H 9050 1100 50  0001 C CNN
+F 1 "GNDREF" H 9055 1177 50  0000 C CNN
+F 2 "" H 9050 1350 50  0001 C CNN
+F 3 "" H 9050 1350 50  0001 C CNN
+	1    9050 1350
+	1    0    0    -1
+$EndComp
+Wire Wire Line
+	9250 1350 9500 1350
+Wire Wire Line
+	9050 1350 9250 1350
+Connection ~ 9250 1350
+$Comp
+L power:GNDREF #PWR?
+U 1 1 5F4AC639
+P 9350 2250
+F 0 "#PWR?" H 9350 2000 50  0001 C CNN
+F 1 "GNDREF" H 9355 2077 50  0000 C CNN
+F 2 "" H 9350 2250 50  0001 C CNN
+F 3 "" H 9350 2250 50  0001 C CNN
+	1    9350 2250
+	1    0    0    -1
+$EndComp
