File: pcb/Micros.kicad_pcb (KiCad board)
At the start: 2 copper layers, 116.8 x 61 mm, 19 parts, among them J1 Conn_02x08, J2 Connector Encoder, J3 Conn_01x10, J4 Conn_01x08, J5 Conn_01x08, J6 Conn_Coaxial, J7 Screw_Terminal_01x02, U1 LMD18200, U2 LS7366R, U3 74LVC1G04

Commit message: Update footprint.
Connections:
- F1 pad 1: +28V -> Net-(F1-Pad1)
- J7 pad 1: +28V -> Net-(J7-Pad1)
- U3 pad 4: Net-(U1-Pad4) -> +5V
- U3 pad 5: +5V -> Net-(U1-Pad4)

Commit message: 3d viewer
Parts:
- moved U3 116.9 mm to (94.7, 133.6), turned to 90 degrees
- moved F1 107.8 mm to (125.8, 129.7), turned to 90 degrees
- moved J1 106.0 mm to (85.9, 152.7), turned to 90 degrees
- moved R2 92.6 mm to (168.8, 131.2), turned to 270 degrees
- moved J7 86.5 mm to (147.6, 140.8)
- moved J4 83.6 mm to (100.6, 142.5), turned to 270 degrees
- moved U1 81.5 mm to (94.9, 124.2)
- moved C4 78.3 mm to (108.2, 104.9), turned to 180 degrees
- moved R1 75.8 mm to (168.0, 116.4)
- moved C3 73.3 mm to (79.9, 123.3), turned to 270 degrees
- moved C1 73.1 mm to (156.5, 107.4)
- moved Crystal1 60.3 mm to (169.0, 103.0)
- moved R3 48.4 mm to (124.2, 113.8)
- moved J6 46.2 mm to (83.1, 107.7)
- moved C2 28.5 mm to (161.6, 122.6)
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Connections:
- F1 pad 1: Net-(F1-Pad1) -> +28V
- J7 pad 1: Net-(J7-Pad1) -> +28V
- U3 pad 4: +5V -> Net-(U1-Pad4)
- U3 pad 5: Net-(U1-Pad4) -> +5V
Routing:
- net GND: track 0.00 -> 139.3 mm
- net +5V: track 0.00 -> 104.6 mm
- net Net-(R2-Pad2): track 0.00 -> 69.0 mm
- net TH_FLAG: track 0.00 -> 44.2 mm
- net Net-(C2-Pad1): track 0.00 -> 40.5 mm
- net Net-(C4-Pad2): track 0.00 -> 34.6 mm
- net Net-(C3-Pad1): track 0.00 -> 30.5 mm
- net Net-(C1-Pad1): track 0.00 -> 29.7 mm
- net Net-(F1-Pad2): track 0.00 -> 25.8 mm
- net +28V: track 0.00 -> 25.4 mm
- net PWM: track 0.00 -> 22.4 mm
- net Net-(C4-Pad1): track 0.00 -> 20.8 mm
- net Net-(C3-Pad2): track 0.00 -> 15.7 mm
- net Net-(U1-Pad4): track 0.00 -> 14.7 mm
- net Net-(J2-Pad5): track 0.00 -> 13.9 mm
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Other:
- board size 116.8 x 61 mm -> 115.6 x 61 mm
