File: pcb/Quanser_Controller.sch (KiCad schematic (older format))
At the start: 19 parts, among them J1 Conn_02x08, J2 Connector Encoder, J3 Conn_01x10, J4 Conn_01x08, J5 Conn_01x08, J6 Screw_Terminal_01x02, J7 Screw_Terminal_01x02, U1 LMD18200, U2 LS7366R, U3 74LVC1G04

Commit message: Update project.
Parts:
- removed U3: 74LVC1G04, Connector_PinHeader_2.00mm:PinHeader_2x03_P2.00mm_Vertical, symbol 74xGxx:74LVC1G04
- added Q1: BC548, Package_TO_SOT_THT:TO-92_Inline, symbol Transistor_BJT:BC548
- added R4: 5K, Resistor_THT:R_Axial_DIN0204_L3.6mm_D1.6mm_P5.08mm_Horizontal, symbol Device:R
- added R5: 2K, Resistor_THT:R_Axial_DIN0204_L3.6mm_D1.6mm_P5.08mm_Horizontal, symbol Device:R
- F1: value 3A -> 5A; footprint Fuse:Fuse_2010_5025Metric_Pad1.52x2.65mm_HandSolder -> Fuse:Fuseholder_Cylinder-5x20mm_Schurter_0031_8201_Horizontal_Open
Connections:
- net labels added: BRAKE, DISABLE
- net labels removed: ENABLE
- wire segments 106 -> 112
- no-connect marks 32 -> 23
Other:
- moved on the sheet: C3, C4, J6, R2, R3, U1

Commit message: Adjust schematic.
Parts:
- added R6, R7: 1K, Resistor_THT:R_Axial_DIN0204_L3.6mm_D1.6mm_P5.08mm_Horizontal, symbol Device:R
- R4: value 5K -> 4K3
- R5: value 2K -> 5K
Connections:
- net +28V: now also F1.1; no longer R5.1
- net +5V: now also R6.1; no longer U1.5 (PWM)
- net GND: now also R5.2, R7.2
- net at U1.6 (VS): now also F1.2; no longer F1.1
- net at Q1.2 (B), R4.1: now also R5.1
- net BRAKE: no longer names the net of U1.4 (BRAKE)
- net BRAKE: now also Q1.1 (C), R6.2; no longer J4.8 (Pin_8)
- net DISABLE renamed ENABLE
- net ENABLE: now also U1.5 (PWM), R7.1
Other:
- moved on the sheet: Q1
Changed lines of the file:
@@
 EESchema Schematic File Version 4
-LIBS:Quanser_Controller-cache
-EELAYER 26 0
+EELAYER 30 0
 EELAYER END
 $Descr A4 11693 8268
@@
 	9450 850  9600 850
 Text GLabel 10450 1150 0    50   Output ~ 0
-DISABLE
+ENABLE
 Wire Wire Line
 	7100 4400 7550 4400
@@
 	7550 4400 7550 4850
 Connection ~ 7100 4400
-Wire Wire Line
-	4500 4800 4500 4750
 $Comp
 L power:+5V #PWR0111
 U 1 1 5F4137B3
-P 4500 4750
-F 0 "#PWR0111" H 4500 4600 50  0001 C CNN
-F 1 "+5V" H 4515 4923 50  0000 C CNN
-F 2 "" H 4500 4750 50  0001 C CNN
-F 3 "" H 4500 4750 50  0001 C CNN
-	1    4500 4750
-	1    0    0    -1
-$EndComp
-Wire Wire Line
-	4500 4800 5000 4800
+P 2600 4900
+F 0 "#PWR0111" H 2600 4750 50  0001 C CNN
+F 1 "+5V" H 2615 5073 50  0000 C CNN
+F 2 "" H 2600 4900 50  0001 C CNN
+F 3 "" H 2600 4900 50  0001 C CNN
+	1    2600 4900
+	1    0    0    -1
+$EndComp
 Wire Wire Line
 	4600 5100 5000 5100
@@
 L Quanser_Controller-rescue:+27V-+27v #PWR0110
 U 1 1 5F54B278
-P 4850 2850
-F 0 "#PWR0110" H 4850 2700 50  0001 C CNN
-F 1 "+27V" H 4850 3023 50  0000 C CNN
-F 2 "" H 5100 2900 50  0001 C CNN
-F 3 "" H 5100 2900 50  0001 C CNN
-	1    4850 2850
+P 5700 3550
+F 0 "#PWR0110" H 5700 3400 50  0001 C CNN
+F 1 "+27V" H 5700 3723 50  0000 C CNN
+F 2 "" H 5950 3600 50  0001 C CNN
+F 3 "" H 5950 3600 50  0001 C CNN
+	1    5700 3550
 	1    0    0    -1
 $EndComp
@@
 L Transistor_BJT:BC548 Q1
 U 1 1 5F4BF13E
-P 4750 3800
-F 0 "Q1" H 4941 3846 50  0000 L CNN
-F 1 "BC548" H 4941 3755 50  0000 L CNN
-F 2 "Package_TO_SOT_THT:TO-92_Inline" H 4950 3725 50  0001 L CIN
-F 3 "http://www.fairchildsemi.com/ds/BC/BC547.pdf" H 4750 3800 50  0001 L CNN
-	1    4750 3800
-	1    0    0    -1
-$EndComp
-$Comp
-L power:GND #PWR0119
-U 1 1 5F4C45FF
-P 4850 4250
-F 0 "#PWR0119" H 4850 4000 50  0001 C CNN
-F 1 "GND" H 4855 4077 50  0000 C CNN
-F 2 "" H 4850 4250 50  0001 C CNN
-F 3 "" H 4850 4250 50  0001 C CNN
-	1    4850 4250
-	1    0    0    -1
-$EndComp
-Wire Wire Line
-	4350 3800 4550 3800
+P 2500 5750
+F 0 "Q1" H 2691 5796 50  0000 L CNN
+F 1 "BC548" H 2691 5705 50  0000 L CNN
+F 2 "Package_TO_SOT_THT:TO-92_Inline" H 2700 5675 50  0001 L CIN
+F 3 "http://www.fairchildsemi.com/ds/BC/BC547.pdf" H 2500 5750 50  0001 L CNN
+	1    2500 5750
+	1    0    0    -1
+$EndComp
+Wire Wire Line
+	5700 3550 5700 3700
+Text GLabel 1350 5750 0    50   Input ~ 0
+ENABLE
+$Comp
+L Device:Fuse F1
+U 1 1 5F50642B
+P 5700 3850
+F 0 "F1" H 5760 3896 50  0000 L CNN
+F 1 "5A" H 5760 3805 50  0000 L CNN
+F 2 "Fuse:Fuseholder_Cylinder-5x20mm_Schurter_0031_8201_Horizontal_Open" V 5630 3850 50  0001 C CNN
+F 3 "~" H 5700 3850 50  0001 C CNN
+	1    5700 3850
+	1    0    0    -1
+$EndComp
+Wire Wire Line
+	5700 4000 5700 4300
+$Comp
+L power:GND #PWR?
+U 1 1 5F586E03
+P 2600 6400
+F 0 "#PWR?" H 2600 6150 50  0001 C CNN
+F 1 "GND" H 2605 6227 50  0000 C CNN
+F 2 "" H 2600 6400 50  0001 C CNN
+F 3 "" H 2600 6400 50  0001 C CNN
+	1    2600 6400
+	1    0    0    -1
+$EndComp
 $Comp
 L Device:R R4
-U 1 1 5F51665F
-P 4200 3800
-F 0 "R4" V 3993 3800 50  0000 C CNN
-F 1 "5K" V 4084 3800 50  0000 C CNN
-F 2 "Resistor_THT:R_Axial_DIN0204_L3.6mm_D1.6mm_P5.08mm_Horizontal" V 4130 3800 50  0001 C CNN
-F 3 "~" H 4200 3800 50  0001 C CNN
-	1    4200 3800
+U 1 1 5F598BC1
+P 1900 5750
+F 0 "R4" V 1693 5750 50  0000 C CNN
+F 1 "4K3" V 1784 5750 50  0000 C CNN
+F 2 "Resistor_THT:R_Axial_DIN0204_L3.6mm_D1.6mm_P5.08mm_Horizontal" V 1830 5750 50  0001 C CNN
+F 3 "~" H 1900 5750 50  0001 C CNN
+	1    1900 5750
 	0    1    1    0
 $EndComp
-Text GLabel 10450 1550 0    50   Output ~ 0
-BRAKE
-Text GLabel 4650 5400 0    50   Input ~ 0
-BRAKE
-Wire Wire Line
-	4850 4000 4850 4250
+Wire Wire Line
+	1350 5750 1750 5750
+Wire Wire Line
+	2050 5750 2200 5750
+Wire Wire Line
+	2600 5400 2600 5550
 $Comp
 L Device:R R5
-U 1 1 5F4FA7EA
-P 4850 3150
-F 0 "R5" H 4920 3196 50  0000 L CNN
-F 1 "2K" H 4920 3105 50  0000 L CNN
-F 2 "Resistor_THT:R_Axial_DIN0204_L3.6mm_D1.6mm_P5.08mm_Horizontal" V 4780 3150 50  0001 C CNN
-F 3 "~" H 4850 3150 50  0001 C CNN
-	1    4850 3150
-	1    0    0    -1
-$EndComp
-Wire Wire Line
-	4850 2850 4850 3000
-Wire Wire Line
-	4850 3300 4850 3450
-Wire Wire Line
-	4650 5400 5000 5400
-$Comp
-L Device:Fuse F1
-U 1 1 5F4EE310
-P 5250 3450
-F 0 "F1" V 5053 3450 50  0000 C CNN
-F 1 "5A" V 5144 3450 50  0000 C CNN
-F 2 "Fuse:Fuseholder_Cylinder-5x20mm_Schurter_0031_8201_Horizontal_Open" V 5180 3450 50  0001 C CNN
-F 3 "~" H 5250 3450 50  0001 C CNN
-	1    5250 3450
-	0    1    1    0
-$EndComp
-Wire Wire Line
-	4850 3450 5100 3450
-Connection ~ 4850 3450
-Wire Wire Line
-	4850 3450 4850 3600
-Wire Wire Line
-	5400 3450 5700 3450
-Wire Wire Line
-	5700 3450 5700 4300
-Text GLabel 3750 3800 0    50   Input ~ 0
-DISABLE
-Wire Wire Line
-	3750 3800 4050 3800
+U 1 1 5F5C9923
+P 2200 6050
+F 0 "R5" H 2270 6096 50  0000 L CNN
+F 1 "5K" H 2270 6005 50  0000 L CNN
+F 2 "Resistor_THT:R_Axial_DIN0204_L3.6mm_D1.6mm_P5.08mm_Horizontal" V 2130 6050 50  0001 C CNN
+F 3 "~" H 2200 6050 50  0001 C CNN
+	1    2200 6050
+	1    0    0    -1
+$EndComp
+Wire Wire Line
+	2600 5950 2600 6300
+Wire Wire Line
+	2200 5750 2200 5900
+Connection ~ 2200 5750
+Wire Wire Line
+	2200 5750 2300 5750
+Wire Wire Line
+	2200 6200 2200 6300
+Wire Wire Line
+	2200 6300 2600 6300
+Connection ~ 2600 6300
+Wire Wire Line
+	2600 6300 2600 6400
+$Comp
+L Device:R R6
+U 1 1 5F5DDD0F
+P 2600 5150
+F 0 "R6" H 2670 5196 50  0000 L CNN
+F 1 "1K" H 2670 5105 50  0000 L CNN
+F 2 "Resistor_THT:R_Axial_DIN0204_L3.6mm_D1.6mm_P5.08mm_Horizontal" V 2530 5150 50  0001 C CNN
+F 3 "~" H 2600 5150 50  0001 C CNN
+	1    2600 5150
+	1    0    0    -1
+$EndComp
+Wire Wire Line
+	2600 4900 2600 5000
+Wire Wire Line
+	2600 5300 2600 5400
+Connection ~ 2600 5400
+Wire Wire Line
+	2600 5400 5000 5400
+Text GLabel 3300 4800 0    50   Input ~ 0
+ENABLE
+$Comp
+L Device:R R7
+U 1 1 5F665EE7
+P 3850 4950
+F 0 "R7" H 3920 4996 50  0000 L CNN
+F 1 "1K" H 3920 4905 50  0000 L CNN
+F 2 "Resistor_THT:R_Axial_DIN0204_L3.6mm_D1.6mm_P5.08mm_Horizontal" V 3780 4950 50  0001 C CNN
+F 3 "~" H 3850 4950 50  0001 C CNN
+	1    3850 4950
+	1    0    0    -1
+$EndComp
+$Comp
+L power:GND #PWR?
+U 1 1 5F68BB45
+P 3850 5150
+F 0 "#PWR?" H 3850 4900 50  0001 C CNN
+F 1 "GND" H 3855 4977 50  0000 C CNN
+F 2 "" H 3850 5150 50  0001 C CNN
+F 3 "" H 3850 5150 50  0001 C CNN
+	1    3850 5150
+	1    0    0    -1
+$EndComp
+Wire Wire Line
+	3850 5100 3850 5150
+Wire Wire Line
+	3850 4800 5000 4800
+Wire Wire Line
+	3300 4800 3850 4800
+Connection ~ 3850 4800
 $EndSCHEMATC

Commit message: update PCB; included reports; add A/D
Parts:
- added AD1: Conn_01x06, Connector_PinHeader_2.00mm:PinHeader_1x06_P2.00mm_Vertical, symbol Connector_Generic:Conn_01x06
Connections:
- net labels added: AD
- wire segments 117 -> 119
Changed lines of the file:
@@
 EESchema Schematic File Version 4
-EELAYER 30 0
+LIBS:Quanser_Controller-cache
+EELAYER 26 0
 EELAYER END
 $Descr A4 11693 8268
@@
 $EndComp
 Wire Wire Line
-	6400 5500 7750 5500
+	6400 5500 7350 5500
 $Comp
 L power:+5V #PWR0113
@@
 	5700 4000 5700 4300
 $Comp
-L power:GND #PWR?
+L power:GND #PWR0119
 U 1 1 5F586E03
 P 2600 6400
-F 0 "#PWR?" H 2600 6150 50  0001 C CNN
+F 0 "#PWR0119" H 2600 6150 50  0001 C CNN
 F 1 "GND" H 2605 6227 50  0000 C CNN
 F 2 "" H 2600 6400 50  0001 C CNN
@@
 $EndComp
 $Comp
-L power:GND #PWR?
+L power:GND #PWR0120
 U 1 1 5F68BB45
 P 3850 5150
-F 0 "#PWR?" H 3850 4900 50  0001 C CNN
+F 0 "#PWR0120" H 3850 4900 50  0001 C CNN
 F 1 "GND" H 3855 4977 50  0000 C CNN
 F 2 "" H 3850 5150 50  0001 C CNN
@@
 	3300 4800 3850 4800
 Connection ~ 3850 4800
+Text GLabel 8200 1100 0    50   Output ~ 0
+AD
+Text GLabel 7350 5700 3    50   Output ~ 0
+AD
+Wire Wire Line
+	7350 5500 7350 5700
+Connection ~ 7350 5500
+Wire Wire Line
+	7350 5500 7750 5500
+$Comp
+L Connector_Generic:Conn_01x06 AD1
+U 1 1 5F510A72
+P 8400 800
+F 0 "AD1" H 8480 746 50  0000 L CNN
+F 1 "Conn_01x06" H 8480 701 50  0001 L CNN
+F 2 "Connector_PinHeader_2.00mm:PinHeader_1x06_P2.00mm_Vertical" H 8400 800 50  0001 C CNN
+F 3 "~" H 8400 800 50  0001 C CNN
+	1    8400 800
+	1    0    0    -1
+$EndComp
 $EndSCHEMATC
