File: pcb/Quanser_Controller.sch (KiCad schematic (older format))
At the start: 24 parts, among them J1 Conn_02x08, J2 Connector Encoder, J3 Conn_01x10, J4 Conn_01x08, J5 Conn_01x08, J6 Screw_Terminal_01x02, J7 Screw_Terminal_01x02, Q1 BC548, U1 LMD18200, U2 LS7366R

Commit message: Last update PCB
Parts:
- removed AD1: Conn_01x06, Connector_PinHeader_2.00mm:PinHeader_1x06_P2.00mm_Vertical, symbol Connector_Generic:Conn_01x06
- added J8: Conn_01x06, Connector_PinHeader_2.00mm:PinHeader_1x06_P2.00mm_Vertical, symbol Connector_Generic:Conn_01x06
Connections:
- net AD: now also J8.6 (Pin_6)
Changed lines of the file:
@@
 EESchema Schematic File Version 4
-EELAYER 30 0
+LIBS:Quanser_Controller-cache
+EELAYER 26 0
 EELAYER END
 $Descr A4 11693 8268
@@
 	3300 4800 3850 4800
 Connection ~ 3850 4800
-Text GLabel 8200 1100 0    50   Output ~ 0
+Text GLabel 7600 1100 0    50   Output ~ 0
 AD
 Text GLabel 7350 5700 3    50   Output ~ 0
@@
 	7350 5500 7750 5500
 $Comp
-L Connector_Generic:Conn_01x06 AD1
-U 1 1 5F510A72
-P 8400 800
-F 0 "AD1" H 8480 746 50  0000 L CNN
-F 1 "Conn_01x06" H 8480 701 50  0001 L CNN
-F 2 "Connector_PinHeader_2.00mm:PinHeader_1x06_P2.00mm_Vertical" H 8400 800 50  0001 C CNN
-F 3 "~" H 8400 800 50  0001 C CNN
-	1    8400 800
-	1    0    0    -1
-$EndComp
+L Connector_Generic:Conn_01x06 J8
+U 1 1 5F542679
+P 7800 800
+F 0 "J8" H 7880 792 50  0000 L CNN
+F 1 "Conn_01x06" H 7880 701 50  0000 L CNN
+F 2 "Connector_PinHeader_2.00mm:PinHeader_1x06_P2.00mm_Vertical" H 7800 800 50  0001 C CNN
+F 3 "~" H 7800 800 50  0001 C CNN
+	1    7800 800
+	1    0    0    -1
+$EndComp

Commit message: included H-Bridge
Connections:
- net TH_FLAG: now also J8.5 (Pin_5); no longer J4.7 (Pin_7)
Changed lines of the file:
@@
 Wire Wire Line
 	6650 6050 6650 6200
-Text GLabel 10450 1450 0    50   Input ~ 0
+Text GLabel 7600 1000 0    50   Input ~ 0
 TH_FLAG
 Wire Wire Line
@@
 	3300 4800 3850 4800
 Connection ~ 3850 4800
-Text GLabel 7600 1100 0    50   Output ~ 0
+Text GLabel 7600 1100 0    50   Input ~ 0
 AD
 Text GLabel 7350 5700 3    50   Output ~ 0
